Commit message: Dual Lidar

File: description/robot_core.xacro (robot description, xacro)
@@ -6,5 +6,5 @@
     <xacro:property name="chassis_height" value="0.9"/>
     <xacro:property name="chassis_mass" value="10.0"/>
-    <xacro:property name="wheel_radius" value="0.172"/>
+    <xacro:property name="wheel_radius" value="0.1592"/>
     <xacro:property name="wheel_thickness" value="0.07"/>
     <xacro:property name="wheel_mass" value="0.05"/>
@@ -42,5 +42,5 @@
         <parent link="base_link"/>
         <child link="base_footprint"/>
-        <origin xyz="0 0 0" rpy="0 0 0"/>
+        <origin xyz="0 0 -${wheel_radius}" rpy="0 0 0"/>
     </joint>
     <link name="base_footprint">
@@ -50,5 +50,5 @@
         <parent link="base_link"/>
         <child link="chassis"/>
-        <origin xyz="-${chassis_length/2} 0.0 -.1"/>
+        <origin xyz="-${chassis_length/2} 0.0 0.0"/>
     </joint>
     <link name="chassis">

File: description/ros2_control.xacro (robot description, xacro)
@@ -11,6 +11,6 @@
                 <state_interface name="position"/>
                 <param name="address">128</param>
-                <param name="qppr">12841</param>
-                <param name="motor_type">M2</param>
+                <param name="qppr">12762</param>
+                <param name="motor_type">M1</param>
             </joint>
             <joint name="right_wheel_joint">
@@ -18,6 +18,6 @@
                 <state_interface name="position"/>
                 <param name="address">128</param>
-                <param name="qppr">12841</param>
-                <param name="motor_type">M1</param>
+                <param name="qppr">12762</param>
+                <param name="motor_type">M2</param>
                 <!-- Add other configurations as necessary -->
             </joint>

File: description/rp_s1_lidar.xacro (robot description, xacro)
@@ -4,5 +4,5 @@
         <parent link="base_link"/>
         <child link="rp_s1_lidar"/>
-        <origin xyz="0.21 0 -0.14" rpy="0 3.145 3.145"/>
+        <origin xyz="0.21 0 0.14" rpy="0 0.0 3.14"/>
     </joint>
     <link name="rp_s1_lidar">

File: description/rp_s2e_lidar.xacro (robot description, xacro)
@@ -4,5 +4,5 @@
         <parent link="base_link"/>
         <child link="rp_s2e_lidar"/>
-        <origin xyz="-0.52 0.0 -0.045" rpy="0.0 0.0 0"/>
+        <origin xyz="-0.52 0.0 0.0" rpy="0.0 0.0 0"/>
     </joint>
     <link name="rp_s2e_lidar">

Commit message: tuning

File: description/robot_core.xacro (robot description, xacro)
@@ -4,5 +4,5 @@
     <xacro:property name="chassis_length" value="0.41"/>
     <xacro:property name="chassis_width" value="0.402"/>
-    <xacro:property name="chassis_height" value="0.9"/>
+    <xacro:property name="chassis_height" value="0.8"/>
     <xacro:property name="chassis_mass" value="10.0"/>
     <xacro:property name="wheel_radius" value="0.1592"/>

File: description/velodyne.xacro (robot description, xacro)
@@ -4,5 +4,5 @@
         <parent link="base_link"/>
         <child link="velodyne_frame"/>
-        <origin xyz="0.140 0.0 0.85" rpy="0 0 0"/>
+        <origin xyz="0.140 0.0 0.8" rpy="0 0 0"/>
     </joint>
     <link name="velodyne_frame">
