Commit message: depth camera

File: description/realsense_d435.xacro (robot description, xacro)
@@ -3,8 +3,8 @@
     <joint name="camera_joint" type="fixed">
         <parent link="chassis"/>
-        <child link="camera_link"/>
-        <origin xyz="0.305 0 0.08" rpy="0 0 0"/>
+        <child link="camera_color_frame"/>
+        <origin xyz="0.24 0 0.08" rpy="0 0 0"/>
     </joint>
-    <link name="camera_link">
+    <link name="camera_color_frame">
         <visual>
             <geometry>
@@ -15,10 +15,10 @@
     </link>
     <joint name="camera_optical_joint" type="fixed">
-        <parent link="camera_link"/>
+        <parent link="camera_color_frame"/>
         <child link="camera_link_optical"/>
         <origin xyz="0 0 0" rpy="${-pi/2} 0 ${-pi/2}"/>
     </joint>
     <link name="camera_link_optical"></link>
-    <gazebo reference="camera_link">
+    <gazebo reference="camera_color_frame">
         <material>Gazebo/Red</material>
         <sensor name="camera" type="depth">

File: description/robot.urdf.xacro (robot description, xacro)
@@ -1,9 +1,9 @@
 <?xml version="1.0"?>
 <robot xmlns:xacro="http://www.ros.org/wiki/xacro"  name="robot">
+<!-- <xacro:include filename="camera.xacro" /> -->
     <xacro:arg name="sim_mode" default="false"/>
     <xacro:include filename="robot_core.xacro" />
     <xacro:include filename="ros2_control.xacro" />
     <xacro:include filename="velodyne.xacro" />
-    <!-- <xacro:include filename="camera.xacro" /> -->
-    <!-- <xacro:include filename="depth_camera.xacro" /> -->
+    <xacro:include filename="realsense_d435.xacro" />
 </robot>

Commit message: local cost map

File: description/realsense_d435.xacro (robot description, xacro)
@@ -2,9 +2,9 @@
 <robot xmlns:xacro="http://www.ros.org/wiki/xacro" >
     <joint name="camera_joint" type="fixed">
-        <parent link="chassis"/>
-        <child link="camera_color_frame"/>
-        <origin xyz="0.24 0 0.08" rpy="0 0 0"/>
+        <parent link="base_link"/>
+        <child link="camera_link"/>
+        <origin xyz="0.24 0 0.18" rpy="0 0 0"/>
     </joint>
-    <link name="camera_color_frame">
+    <link name="camera_link">
         <visual>
             <geometry>
@@ -15,10 +15,10 @@
     </link>
     <joint name="camera_optical_joint" type="fixed">
-        <parent link="camera_color_frame"/>
+        <parent link="camera_link"/>
         <child link="camera_link_optical"/>
         <origin xyz="0 0 0" rpy="${-pi/2} 0 ${-pi/2}"/>
     </joint>
     <link name="camera_link_optical"></link>
-    <gazebo reference="camera_color_frame">
+    <gazebo reference="camera_link">
         <material>Gazebo/Red</material>
         <sensor name="camera" type="depth">

Commit message: dual slamtech lidars, realsense

File: description/realsense_d435.xacro (robot description, xacro)
@@ -4,5 +4,5 @@
         <parent link="base_link"/>
         <child link="camera_link"/>
-        <origin xyz="0.24 0 0.18" rpy="0 0 0"/>
+        <origin xyz="-0.24 0 0.18" rpy="0 0 3.14"/>
     </joint>
     <link name="camera_link">

File: description/robot.urdf.xacro (robot description, xacro)
@@ -6,4 +6,6 @@
     <xacro:include filename="ros2_control.xacro" />
     <xacro:include filename="velodyne.xacro" />
+    <xacro:include filename="rp_s1_lidar.xacro" />
+    <xacro:include filename="rp_s2e_lidar.xacro" />
     <xacro:include filename="realsense_d435.xacro" />
 </robot>

File: description/robot_core.xacro (robot description, xacro)
@@ -29,4 +29,7 @@
         <color rgba="0 0 0 1"/>
     </material>
+    <material name="gray">
+        <color rgba="0 0 0 0.5"/>
+    </material>
     <material name="red">
         <color rgba="1 0 0 1"/>

File: description/rp_s1_lidar.xacro (robot description, xacro)
@@ -1,35 +1,35 @@
 <?xml version="1.0"?>
 <robot xmlns:xacro="http://www.ros.org/wiki/xacro" >
-    <joint name="velodyne_joint" type="fixed">
+    <joint name="rp_s1_lidar_joint" type="fixed">
         <parent link="base_link"/>
-        <child link="velodyne_frame"/>
-        <origin xyz="0.140 0.0 0.85" rpy="0 0 0"/>
+        <child link="rp_s1_lidar"/>
+        <origin xyz="0.21 0 -0.14" rpy="0 3.145 3.145"/>
     </joint>
-    <link name="velodyne_frame">
+    <link name="rp_s1_lidar">
         <visual>
             <geometry>
-                <cylinder radius="0.072" length="0.103"/>
+                <cylinder radius="0.03" length="0.03"/>
             </geometry>
             <material name="black"/>
         </visual>
         <visual>
-            <origin xyz="0 0 -0.05"/>
+            <origin xyz="0 0 -0.03"/>
             <geometry>
-                <cylinder radius="0.01" length="0.1"/>
+                <cylinder radius="0.03" length="0.03"/>
             </geometry>
-            <material name="black"/>
+            <material name="gray"/>
         </visual>
         <collision>
             <geometry>
-                <cylinder radius="0.05" length="0.04"/>
+                <cylinder radius="0.03" length="0.02"/>
             </geometry>
         </collision>
-        <xacro:inertial_cylinder mass="0.1" length="0.04" radius="0.05">
+        <xacro:inertial_cylinder mass="0.1" length="0.02" radius="0.03">
             <origin xyz="0 0 0" rpy="0 0 0"/>
         </xacro:inertial_cylinder>
     </link>
-    <gazebo reference="velodyne_frame">
+    <gazebo reference="rp_s1_lidar">
         <material>Gazebo/Black</material>
-        <sensor name="velodyne" type="ray">
+        <sensor name="laser" type="ray">
             <pose> 0 0 0 0 0 0 </pose>
             <visualize>false</visualize>
@@ -44,14 +44,14 @@
                 </scan>
                 <range>
-                    <min>0.1</min>
-                    <max>25</max>
+                    <min>0.3</min>
+                    <max>12</max>
                 </range>
             </ray>
-            <plugin name="velodyne_controller" filename="libgazebo_ros_ray_sensor.so">
+            <plugin name="laser_controller" filename="libgazebo_ros_ray_sensor.so">
                 <ros>
-                    <argument>~/out:=scan</argument>
+                    <argument>~/out:=rp_s1_lidar/scan</argument>
                 </ros>
                 <output_type>sensor_msgs/LaserScan</output_type>
-                <frame_name>velodyne_frame</frame_name>
+                <frame_name>rp_s1_lidar</frame_name>
             </plugin>
         </sensor>

File: description/rp_s2e_lidar.xacro (robot description, xacro)
@@ -1,20 +1,20 @@
 <?xml version="1.0"?>
 <robot xmlns:xacro="http://www.ros.org/wiki/xacro" >
-    <joint name="laser_joint" type="fixed">
-        <parent link="chassis"/>
-        <child link="laser_frame"/>
-        <origin xyz="0.122 0 0.212" rpy="0 0 0"/>
+    <joint name="rp_s2e_lidar_joint" type="fixed">
+        <parent link="base_link"/>
+        <child link="rp_s2e_lidar"/>
+        <origin xyz="-0.52 0.0 -0.045" rpy="0.0 0.0 0"/>
     </joint>
-    <link name="laser_frame">
+    <link name="rp_s2e_lidar">
         <visual>
             <geometry>
-                <cylinder radius="0.05" length="0.04"/>
+                <cylinder radius="0.05" length="0.03"/>
             </geometry>
-            <material name="black"/>
+            <material name="gray"/>
         </visual>
         <visual>
-            <origin xyz="0 0 -0.05"/>
+            <origin xyz="0 0 -0.03"/>
             <geometry>
-                <cylinder radius="0.01" length="0.1"/>
+                <cylinder radius="0.05" length="0.03"/>
             </geometry>
             <material name="black"/>
@@ -22,5 +22,5 @@
         <collision>
             <geometry>
-                <cylinder radius="0.05" length="0.04"/>
+                <cylinder radius="0.05" length="0.06"/>
             </geometry>
         </collision>
@@ -29,5 +29,5 @@
         </xacro:inertial_cylinder>
     </link>
-    <gazebo reference="laser_frame">
+    <gazebo reference="rp_s2e_lidar">
         <material>Gazebo/Black</material>
         <sensor name="laser" type="ray">
@@ -50,8 +50,8 @@
             <plugin name="laser_controller" filename="libgazebo_ros_ray_sensor.so">
                 <ros>
-                    <argument>~/out:=scan</argument>
+                    <argument>~/out:=rp_s2e_lidar/scan</argument>
                 </ros>
                 <output_type>sensor_msgs/LaserScan</output_type>
-                <frame_name>laser_frame</frame_name>
+                <frame_name>rp_s2e_lidar</frame_name>
             </plugin>
         </sensor>

Commit message: through door

File: description/realsense_d435.xacro (robot description, xacro)
@@ -4,5 +4,5 @@
         <parent link="base_link"/>
         <child link="camera_link"/>
-        <origin xyz="-0.24 0 0.18" rpy="0 0 3.14"/>
+        <origin xyz="0.24 0 0.18" rpy="0 -0.8 0"/>
     </joint>
     <link name="camera_link">
